File: PJ-005-B/charge amp & inverting amp.kicad_sch (KiCad schematic)
At the start: 16 parts, among them U12 AD8608ARUZ-REEL, U13 TLV365QDBVRQ1

Commit message: -- Receive stage with charge amp-->inverting amp-->BPF-->inverting amp-->buffer-->PGA-->buffer -- Transmit stage with push pull mosfet -- TTL to RS485 converter -- LDOs 12V to 9V, 9V to 6V, 6V to 5V, 5V to 2.5V and -5V to -2.5V
Parts:
- added TP4, TP5: TestPoint, TestPoint:TestPoint_Pad_1.0x1.0mm, symbol Connector:TestPoint
- C25: renamed from C53; footprint (none) -> XaltenFootprints:C0603
- C26: renamed from C54; footprint (none) -> XaltenFootprints:C0603
- C27: renamed from C35; footprint (none) -> XaltenFootprints:C0603
- C28: renamed from C55; footprint (none) -> XaltenFootprints:C0603
- C29: renamed from C36; footprint (none) -> XaltenFootprints:C0603
- C30: renamed from C50; footprint (none) -> XaltenFootprints:C0603
- C31: renamed from C51; footprint (none) -> XaltenFootprints:C0603
- C32: renamed from C34; footprint (none) -> XaltenFootprints:C0603
- C33: renamed from C52; footprint (none) -> XaltenFootprints:C0603
- R28: renamed from R35; value R -> 33R,1%; footprint (none) -> XaltenFootprints:R0603
- R29: renamed from R36; value R -> 3K3,1%; footprint (none) -> XaltenFootprints:R0603
- R30: renamed from R37; footprint (none) -> XaltenFootprints:R0603
- R31: renamed from R33; footprint (none) -> XaltenFootprints:R0603
- R32: renamed from R34; footprint (none) -> XaltenFootprints:R0603
- U10: renamed from U12; footprint (none) -> Echosounder Transceiver FP:RU_14_ADI-L
- U9: renamed from U13; footprint (none) -> XaltenFootprints:SOT-23-5
Connections:
- net +3.3V: now also U10.4 (V+)
- net at C27.2, R29.2, R30.1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: now also TP4.1
- net at C29.1, R30.2: now also TP5.1
Other:
- note added: "Charge Amplifier + Inverting Amplifier (10dB)"
- moved on the sheet: C27, C29, C32, R28, R29, R30, R31, R32, U10A, U9

Commit message: Transceiver After Review
-- Added bulk capacitors for -2.5V LDO
-- Added 0R for shorting RE and DE in TTL to RS485
-- Changed the snubber values in transformer primary to 2.2nF and 33R
-- Removed the 10nF and 100K in parallel with the transducer
-- Added 1000uF capacitor for transformer centre tap
-- Added 100pF decoupling capacitor for gate driver IC
--Changed secondary snubber values to 220nF and 680R
-- Changed LC inductor value to 100uH (transformer secondary)
Parts:
- added J9: Conn_01x02_Pin, Connector_PinHeader_2.54mm:PinHeader_1x02_P2.54mm_Vertical, symbol Connector:Conn_01x02_Pin
Connections:
- net GND: now also J9.1 (Pin_1)
- net at C27.2, R29.2, R30.1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: now also J9.2 (Pin_2)
Changed lines of the file:
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@@
+	)
+	(junction
+		(at 137.16 68.58)
+		(diameter 0)
+		(color 0 0 0 0)
 	)
 	(junction
@@
 		(color 0 0 0 0)
 	)
+	(wire
+		(pts
+			(xy 137.16 68.58) (xy 139.7 68.58)
+		)
+		(stroke
+			(width 0)
+			(type default)
+		)
+	)
 	(polyline
 		(pts
@@
 	(wire
 		(pts
+			(xy 137.16 83.82) (xy 148.59 83.82)
+		)
+		(stroke
+			(width 0)
+			(type default)
+		)
+	)
+	(wire
+		(pts
 			(xy 93.98 130.81) (xy 93.98 135.89)
 		)
@@
 	(wire
 		(pts
+			(xy 148.59 81.28) (xy 137.16 81.28)
+		)
+		(stroke
+			(width 0)
+			(type default)
+		)
+	)
+	(wire
+		(pts
 			(xy 130.81 68.58) (xy 135.89 68.58)
 		)
@@
 	(wire
 		(pts
+			(xy 137.16 86.36) (xy 137.16 83.82)
+		)
+		(stroke
+			(width 0)
+			(type default)
+		)
+	)
+	(wire
+		(pts
 			(xy 113.03 58.42) (xy 113.03 62.23)
 		)
@@
 	(wire
 		(pts
-			(xy 135.89 68.58) (xy 139.7 68.58)
+			(xy 135.89 68.58) (xy 137.16 68.58)
 		)
 		(stroke
@@
 		(pts
 			(xy 135.89 57.15) (xy 135.89 68.58)
+		)
+		(stroke
+			(width 0)
+			(type default)
+		)
+	)
+	(wire
+		(pts
+			(xy 137.16 81.28) (xy 137.16 68.58)
 		)
 		(stroke
@@
 			)
 			(justify left)
+		)
+	)
+	(symbol
+		(lib_id "Connector:Conn_01x02_Pin")
+		(at 153.67 83.82 180)
+		(unit 1)
+		(exclude_from_sim no)
+		(in_bom yes)
+		(on_board yes)
+		(dnp no)
+		(fields_autoplaced yes)
+		(property "Reference" "J9"
+			(at 154.94 81.2799 0)
+			(effects
+				(font
+					(size 1.27 1.27)
+				)
+				(justify right)
+			)
+		)
+		(property "Value" "Conn_01x02_Pin"
+			(at 154.94 83.8199 0)
+			(effects
+				(font
+					(size 1.27 1.27)
+				)
+				(justify right)
+			)
+		)
+		(property "Footprint" "Connector_PinHeader_2.54mm:PinHeader_1x02_P2.54mm_Vertical"
+			(at 153.67 83.82 0)
+			(effects
+				(font
+					(size 1.27 1.27)
+				)
+				(hide yes)
+			)
+		)
+		(property "Datasheet" "~"
+			(at 153.67 83.82 0)
+			(effects
+				(font
+					(size 1.27 1.27)
+				)
+				(hide yes)
+			)
+		)
+		(property "Description" "Generic connector, single row, 01x02, script generated"
+			(at 153.67 83.82 0)
+			(effects
+				(font
+					(size 1.27 1.27)
+				)
+				(hide yes)
+			)
+		)
+		(pin "2"
+		)
+		(pin "1"
+		)
+		(instances
+			(project ""
+				(path "/f8bcf36d-3331-4358-bdb9-a545dbff75f1/e46ac39f-11d3-485e-813c-632dbc6a3109/719e498a-c24a-45e1-9915-628fc4e9a290"
+					(reference "J9")
+					(unit 1)
+				)
+			)
 		)
 	)
@@
 	)
 	(symbol
+		(lib_id "power:GND")
+		(at 137.16 86.36 0)
+		(unit 1)
+		(exclude_from_sim no)
+		(in_bom yes)
+		(on_board yes)
+		(dnp no)
+		(property "Reference" "#PWR0104"
+			(at 137.16 92.71 0)
+			(effects
+				(font
+					(size 1.27 1.27)
+				)
+				(hide yes)
+			)
+		)
+		(property "Value" "GND"
+			(at 139.7 86.36 0)
+			(effects
+				(font
+					(size 1.27 1.27)
+				)
+			)
+		)
+		(property "Footprint" ""
+			(at 137.16 86.36 0)
+			(effects
+				(font
+					(size 1.27 1.27)
+				)
+				(hide yes)
+			)
+		)
+		(property "Datasheet" ""
+			(at 137.16 86.36 0)
+			(effects
+				(font
+					(size 1.27 1.27)
+				)
+				(hide yes)
+			)
+		)
+		(property "Description" "Power symbol creates a global label with name \"GND\" , ground"
+			(at 137.16 86.36 0)
+			(effects
+				(font
+					(size 1.27 1.27)
+				)
+				(hide yes)
+			)
+		)
+		(pin "1"
+		)
+		(instances
+			(project "PJ-005-B"
+				(path "/f8bcf36d-3331-4358-bdb9-a545dbff75f1/e46ac39f-11d3-485e-813c-632dbc6a3109/719e498a-c24a-45e1-9915-628fc4e9a290"
+					(reference "#PWR0104")
+					(unit 1)
+				)
+			)
+		)
+	)
+	(symbol
 		(lib_id "Device:C")
 		(at 215.9 127 180)
@@
 		(dnp no)
 		(property "Reference" "U9"
-			(at 129.54 62.1598 0)
+			(at 107.696 60.96 0)
 			(effects
 				(font
@@
 		)
 		(property "Value" "TLV365QDBVRQ1"
-			(at 121.412 60.706 0)
+			(at 122.936 72.39 0)
 			(effects
 				(font
@@
 		(dnp no)
 		(property "Reference" "U10"
-			(at 219.71 64.6998 0)
+			(at 197.866 62.992 0)
 			(effects
 				(font
@@
 		)
 		(property "Value" "AD8608ARUZ-REEL"
-			(at 216.916 68.072 0)
-			(effects
-				(font
+			(at 215.646 73.914 0)
+			(effects
+				(font
