File: PJ-005-B/pga.kicad_sch (KiCad schematic)
At the start: 0 parts

Commit message: -- Receive stage with charge amp-->inverting amp-->BPF-->inverting amp-->buffer-->PGA-->buffer -- Transmit stage with push pull mosfet -- TTL to RS485 converter -- LDOs 12V to 9V, 9V to 6V, 6V to 5V, 5V to 2.5V and -5V to -2.5V
Parts:
- added C49: 1uF,16V, XaltenFootprints:C0603, symbol Device:C
- added C50: 2.2uF,25V, XaltenFootprints:C0603, symbol Device:C
- added C51: 100nF,25V, XaltenFootprints:C0603, symbol Device:C
- added C52: 100pF,25V, XaltenFootprints:C0603, symbol Device:C
- added C53: 2pF,25V, XaltenFootprints:C0603, symbol Device:C
- added J5: Pin Header 3 Pin, Connector_PinHeader_2.54mm:PinHeader_1x03_P2.54mm_Vertical, symbol Connector:Conn_01x03_Pin
- added J6: Conn_01x02_Pin, Connector_JST:JST_XH_B2B-XH-A_1x02_P2.50mm_Vertical, symbol Connector:Conn_01x02_Pin
- added R57, R58: 10R,1%, XaltenFootprints:R0603, symbol Device:R
- added R59: 4K7,1%, XaltenFootprints:R0603, symbol Device:R
- added R60, R61: 0R, XaltenFootprints:R0603, symbol Device:R
- added R62, R63: 1K,1%, XaltenFootprints:R0603, symbol Device:R
- added TP17, TP18: TestPoint, TestPoint:TestPoint_Pad_1.0x1.0mm, symbol Connector:TestPoint
- added U10: AD8608ARUZ-REEL, Echosounder Transceiver FP:RU_14_ADI-L, symbol Echosounder Transceiver:AD8608ARUZ-REEL
- added U12: MCP6S91-E/MS, Echosounder Transceiver FP:MSOP8, symbol Echosounder Transceiver:MCP6S91-E_MS
Connections:
- new net: R60.2, R61.2, R62.1, TP18.1
- new net: R61.1, TP17.1, U12.1 (VOUT)
- new net: C49.2, U12.2 (CH0)
- new net: C53.1, R62.2, R63.1, U10.13 (-IND)
- new net: C53.2, J6.2 (Pin_2), R63.2, U10.14 (OUTD)
- new net: J5.2 (Pin_2), R57.1
- new net: J5.3 (Pin_3), R58.1
- new net +3.3V: C50.2, C51.1, C52.1, R59.1, U10.4 (V+), U12.8 (VDD)
- new net CS: J5.1 (Pin_1), R59.2, U12.5 (CS)
- new net GND: C50.1, C51.2, C52.2, J6.1 (Pin_1), U10.11 (V-), U12.4 (VSS)
- new net PGA_IN: C49.1, R60.1
- new net SCK: R58.2, U12.7 (SCK)
- new net SI: R57.2, U12.6 (SI)
- new net VREF: U10.12 (+IND), U12.3 (VREF)
Other:
- note added: "Programmable Gain Amplifier (1, 2, 4, 5, 8, 10, 16, 32 V/V)"

Commit message: Transceiver After Review
-- Added bulk capacitors for -2.5V LDO
-- Added 0R for shorting RE and DE in TTL to RS485
-- Changed the snubber values in transformer primary to 2.2nF and 33R
-- Removed the 10nF and 100K in parallel with the transducer
-- Added 1000uF capacitor for transformer centre tap
-- Added 100pF decoupling capacitor for gate driver IC
--Changed secondary snubber values to 220nF and 680R
-- Changed LC inductor value to 100uH (transformer secondary)
Changed lines of the file:
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@@
 		(on_board yes)
 		(dnp no)
-		(fields_autoplaced yes)
 		(property "Reference" "U12"
-			(at 144.78 101.6 0)
+			(at 124.714 111.76 0)
 			(effects
 				(font
@@
 		)
 		(property "Value" "MCP6S91-E/MS"
-			(at 144.78 104.14 0)
+			(at 135.636 122.428 0)
 			(effects
 				(font
@@
 		(on_board yes)
 		(dnp no)
-		(fields_autoplaced yes)
 		(property "Reference" "U10"
-			(at 236.22 107.8798 0)
+			(at 214.63 106.934 0)
 			(effects
 				(font
@@
 		)
 		(property "Value" "AD8608ARUZ-REEL"
-			(at 236.22 110.4198 0)
-			(effects
-				(font
+			(at 231.648 117.856 0)
+			(effects
+				(font
