File: PJ-005-B/transmit.kicad_sch (KiCad schematic)
At the start: 0 parts

Commit message: Transmitter
-- Preamp 9.5dB gain
-- Power amp 6dB gain
Parts:
- added C10, C13: C, XaltenFootprints:C0603, symbol Device:C
- added C11, C12, C14, C15, C16, C20, C21, C24, C25, C28, C29, C32, C33, C9: 100nF,25V, XaltenFootprints:C0603, symbol Device:C
- added C17: 1uF,25V, XaltenFootprints:C0603, symbol Device:C
- added C18, C19, C22, C23: 6.8uF,25V, XaltenFootprints:C0603, symbol Device:C_Polarized
- added C26, C27, C30, C31: 4.7uF,25V, XaltenFootprints:C0603, symbol Device:C_Polarized
- added J1: Conn_01x02_Pin, Connector_JST:JST_XH_B2B-XH-A_1x02_P2.50mm_Vertical, symbol Connector:Conn_01x02_Pin
- added J2: Conn_01x03_Pin, Connector_JST:JST_XH_B3B-XH-A_1x03_P2.50mm_Vertical, symbol Connector:Conn_01x03_Pin
- added Q1, Q2: Q_NMOS_GSD, XaltenFootprints:SOT-23-3, symbol Transistor_FET:Q_NMOS_GSD
- added R10, R15, R22: 33K,1%, XaltenFootprints:R0603, symbol Device:R
- added R11, R12, R13, R14, R18, R21, R9: 1K,1%, XaltenFootprints:R0603, symbol Device:R
- added R16, R17, R23, R24: 576R,1%, XaltenFootprints:R0603, symbol Device:R
- added R19, R20: 1K5,1%, XaltenFootprints:R0603, symbol Device:R
- added R25, R26, R31, R32: 0R, XaltenFootprints:R0603, symbol Device:R
- added R27, R28, R29, R30: 10K,1%, XaltenFootprints:R0603, symbol Device:R
- added U10: B65821C1008T1, Echosounder Transceiver FP:RM6, symbol Echosounder Transceiver:B65821C1008T1
- added U6, U7: LM7171AIMX/NOPB, XaltenFootprints:SOIC-8-5.3x5.3x1.27, symbol Echosounder Transceiver:LM7171AIMX/NOPB
- added U8, U9: LT1210CR-PBF, Echosounder Transceiver FP:DDPAK-7, symbol Echosounder Transceiver:LT1210CR-PBF
Connections:
- new net: C10.1, R11.1, R13.2, U6.2 (-IN)
- new net: R10.2, R9.2, U6.3 (+IN)
- new net: C10.2, C11.1, R12.2, U6.6 (OUT)
- new net: C16.2, R23.2, R26.1, U9.7 (OUT)
- new net: R26.2, U10.4
- new net: Q1.1 (G), R28.1, R31.2
- new net: C12.2, R18.1
- new net: C13.1, R18.2, R19.1, U7.2 (-IN)
- new net: Q2.1 (G), R29.1, R32.2
- new net: C17.1, U10.3
- new net: C17.2, U10.2
- new net: R16.1, R17.2, U8.1 (-IN)
- new net: C15.2, R16.2, R25.1, U8.7 (OUT)
- new net: R25.2, U10.1
- new net: C14.2, R21.1
- new net: R21.2, R22.2, U9.2 (+IN)
- new net: C12.1, C9.1, J1.2 (Pin_2)
- new net: C16.1, U9.5 (COMP)
- new net: R19.2, R20.1
- new net: C13.2, C14.1, R20.2, U7.6 (OUT)
- new net: R14.2, R15.2, U8.2 (+IN)
- new net: C15.1, U8.5 (COMP)
- new net: R23.1, R24.2, U9.1 (-IN)
- new net: C9.2, R9.1
- new net: R11.2, R12.1
- new net: C11.2, R14.1
- new net +12V: C18.1, C20.1, C22.1, C24.1, C26.1, C28.1, C30.1, C32.1, R27.1, R30.1, U6.7 (V+), U7.7 (V+), U8.4 (V+)
- new net -12V: C19.1, C21.2, C23.1, C25.2, C27.1, C29.2, C31.1, C33.2, U6.4 (V-), U7.4 (V-), U8.6 (V-), U9.6 (V-)
- new net GND: C18.2, C19.2, C20.2, C21.1, C22.2, C23.2, C24.2, C25.1, C26.2, C27.2, C28.2, C29.1, C30.2, C31.2, C32.2, C33.1, J1.1 (Pin_1), J2.2 (Pin_2), Q1.2 (S), Q2.2 (S), R10.1, R13.1, R15.1, R17.1, R22.1, R24.1, R28.2, R29.2, U7.3 (+IN)
- new net SD1: Q1.3 (D), R27.2, U8.3 (SD)
- new net SD2: Q2.3 (D), R30.2, U9.3 (SD)
- new net SHDN1: J2.1 (Pin_1), J2.3 (Pin_3), R31.1, R32.1
Other:
- note added: "Power Amp"
- note added: "Preamp"
- note added: "Preamp (9.5dB) + Power amp (6dB)"
- note added: "Shutdown"
- note added: "Shutdown Active High"

Commit message: -- Transmitter with pre-amp LM7171 and power amp LT1210 -- Receiver with charge amp-->inverting amp-->4th order filter-->Inverting amp-->buffer -- Power with LDO 12V to 9V, 9V to 6V, 6V to 5V, 5V to 2.5V and -5V to -2.5V
Other:
- company: (none) -> Xalten Systems Pvt. Ltd.
- title: (none) -> Echosounder Transceiver
Changed lines of the file:
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@@
 	(generator_version "9.0")
 	(paper "A2")
+	(title_block
+		(title "Echosounder Transceiver")
+		(date "06-04-2026")
+		(rev "0.1")
+		(company "Xalten Systems Pvt. Ltd.")
+		(comment 1 "Designed by: Varun G")
+	)
 	(text "Shutdown"
 		(exclude_from_sim no)

Commit message: -- Receive stage with charge amp-->inverting amp-->BPF-->inverting amp-->buffer-->PGA-->buffer -- Transmit stage with push pull mosfet -- TTL to RS485 converter -- LDOs 12V to 9V, 9V to 6V, 6V to 5V, 5V to 2.5V and -5V to -2.5V
Parts:
- removed C10, C13: C, XaltenFootprints:C0603, symbol Device:C
- removed C11, C12, C14, C15, C25, C28, C29, C32, C33, C9: 100nF,25V, XaltenFootprints:C0603, symbol Device:C
- removed C18, C19, C22, C23: 6.8uF,25V, XaltenFootprints:C0603, symbol Device:C_Polarized
- removed C26, C27, C30, C31: 4.7uF,25V, XaltenFootprints:C0603, symbol Device:C_Polarized
- removed J1: Conn_01x02_Pin, Connector_JST:JST_XH_B2B-XH-A_1x02_P2.50mm_Vertical, symbol Connector:Conn_01x02_Pin
- removed J2: Conn_01x03_Pin, Connector_JST:JST_XH_B3B-XH-A_1x03_P2.50mm_Vertical, symbol Connector:Conn_01x03_Pin
- removed Q1, Q2: Q_NMOS_GSD, XaltenFootprints:SOT-23-3, symbol Transistor_FET:Q_NMOS_GSD
- removed R10: 33K,1%, XaltenFootprints:R0603, symbol Device:R
- removed R11, R12, R13, R14, R9: 1K,1%, XaltenFootprints:R0603, symbol Device:R
- removed R28, R29, R30: 10K,1%, XaltenFootprints:R0603, symbol Device:R
- removed R31, R32: 0R, XaltenFootprints:R0603, symbol Device:R
- removed U10: B65821C1008T1, Echosounder Transceiver FP:RM6, symbol Echosounder Transceiver:B65821C1008T1
- removed U6, U7: LM7171AIMX/NOPB, XaltenFootprints:SOIC-8-5.3x5.3x1.27, symbol Echosounder Transceiver:LM7171AIMX/NOPB
- removed U8, U9: LT1210CR-PBF, Echosounder Transceiver FP:DDPAK-7, symbol Echosounder Transceiver:LT1210CR-PBF
- added C15: 4.7uF,25V, XaltenFootprints:C1206, symbol Device:C_Polarized
- added C18: 100nF,25V, XaltenFootprints:C0603, symbol Device:C
- added C19: 3.9nF,25V, XaltenFootprints:C0603, symbol Device:C
- added C22, C23: 22nF,200V, XaltenFootprints:C0603, symbol Device:C
- added D10, D11, D8, D9: AU1PMHM3_84A, Echosounder Transceiver FP:AU1PMHM384A, symbol Device:D
- added D6, D7: 1N4148W, XaltenFootprints:SOD-123, symbol Device:D
- added IC1: 2EDN8534FXTMA1, Echosounder Transceiver FP:SOIC127P602X173-8N, symbol Echosounder Transceiver:2EDN8534FXTMA1
- added J3: Pin Header 4 Pin, Connector_PinHeader_2.54mm:PinHeader_1x04_P2.54mm_Vertical, symbol Connector:Conn_01x04_Pin
- added J4: 3 Pin JST XH, Connector_JST:JST_XH_B3B-XH-A_1x03_P2.50mm_Vertical, symbol Connector:Conn_01x03_Pin
- added L1: 33uH,840mA, Echosounder Transceiver FP:INDPM4040X300N, symbol Device:L
- added Q1, Q2: SIR622DP-T1-RE3, Echosounder Transceiver FP:SIR622DPT1RE3, symbol Simulation_SPICE:NMOS
- added U8: B65821C1008T1, Echosounder Transceiver FP:RM6, symbol Echosounder Transceiver:B65821C1008T1
- C17: value 1uF,25V -> 100nF,25V
- C20: value 100nF,25V -> 3.9nF,25V
- C21, C24: value 100nF,25V -> 10nF,200V
- R15: value 33K,1% -> 10K,1%
- R16, R17: value 576R,1% -> 10K,1%
- R18: value 1K,1% -> 10K,1%
- R19: value 1K5,1% -> 4R7,1%
- R20: value 1K5,1% -> 2R2,1%
- R21: value 1K,1% -> 4R7,1%
- R22: value 33K,1% -> 2R2,1%
- R23, R24: value 576R,1% -> 12R,1%
- R25: value 0R -> 330R,1%
- R26: value 0R -> 2R5,1%
- R27: value 10K,1% -> 100K,1%
Connections:
- net -12V is gone; now on an unnamed net: C21.2
- net SD1 is gone; now on net GND: R27.2
- net +12V: now also C16.2, C17.1, C15.1, C18.1, IC1.6 (VDD), U8.2, U8.3; no longer C20.1, C24.1, R27.1
- net GND: now also C16.1, C17.2, R15.2, R16.2, R18.2, R23.2, R25.1, C15.2, C18.2, C23.2, IC1.3 (GND), J4.1 (Pin_1), J4.2 (Pin_2), Q1.2 (S), Q2.2 (S), U8.5; no longer C20.2, C21.1, R15.1, R22.1
- net TxD_P: now reaches R26.2
- net TxD_P: now also C24.1, R27.1, J4.3 (Pin_3)
- net PWM_OUT_B: now reaches R18.1
- net PWM_OUT_B: now also R21.1, D7.1 (K), IC1.5 (OUTB)
- net PWM_OUT_A: now reaches R19.1
- net PWM_OUT_A: now also R17.2, D6.1 (K), IC1.7 (OUTA); no longer R18.2
- net EN_A: now reaches R16.1
- net EN_A: now also IC1.1 (ENA), J3.3 (Pin_3); no longer R17.2
- net at R21.2, R22.2: now also Q2.1 (G)
- net at R20.1: now also D6.2 (A); no longer R19.2
- net at R20.2: now also R19.2, Q1.1 (G)
- net at R23.1: now also C19.1; no longer R24.2
- new net: D7.2 (A), R22.1
- new net: D10.2 (A), D11.1 (K), D8.1 (K), D9.2 (A)
- new net: C22.1, D8.2 (A), D9.1 (K), L1.2
- new net: C19.2, Q1.3 (D), U8.1
- new net: C20.1, Q2.3 (D), U8.4
- new net: C21.1, L1.1, U8.8
- new net: D10.1 (K), D11.2 (A), R26.1
- new net: C20.2, R24.2
- new net: C22.2, C23.1
- new net EN_B: IC1.8 (ENB), J3.4 (Pin_4), R15.1
- new net PWM_IN_A: IC1.2 (INA), J3.1 (Pin_1)
- new net PWM_IN_B: IC1.4 (INB), J3.2 (Pin_2)
- no-connect marks 0 -> 2
Other:
- note added: "Gate Driver"
- note added: "Push Pull Stage"
- note added: "Transducer"
- note added: "Transformer RM6"
- note removed: "Power Amp"
- note removed: "Preamp"
- note removed: "Preamp (9.5dB) + Power amp (6dB)"
- note removed: "Shutdown"
- note removed: "Shutdown Active High"

Commit message: Transceiver After Review
-- Added bulk capacitors for -2.5V LDO
-- Added 0R for shorting RE and DE in TTL to RS485
-- Changed the snubber values in transformer primary to 2.2nF and 33R
-- Removed the 10nF and 100K in parallel with the transducer
-- Added 1000uF capacitor for transformer centre tap
-- Added 100pF decoupling capacitor for gate driver IC
--Changed secondary snubber values to 220nF and 680R
-- Changed LC inductor value to 100uH (transformer secondary)
Parts:
- removed C24: 10nF,200V, XaltenFootprints:C0603, symbol Device:C
- removed R27: 100K,1%, XaltenFootprints:R0603, symbol Device:R
- added C57: 100pF,25V, XaltenFootprints:C0603, symbol Device:C
- added C58: 1000uF,35V, Capacitor_THT:CP_Radial_D8.0mm_P3.50mm, symbol Device:C_Polarized
- C19, C20: value 3.9nF,25V -> 2.2nF,50V
- C21: value 10nF,200V -> 220pF,400V
- L1: value 33uH,840mA -> 100uH,840mA
- R23, R24: value 12R,1% -> 33R,1%
- R25: value 330R,1% -> 680R,1%,500mW
Connections:
- net +12V: now also C57.2, C58.1
- net GND: now also C57.1, C58.2
Other:
- moved on the sheet: C15, C16, D10, D11, D8, D9, R26
